File: psu-pcb/psu.sch (EAGLE design)
At the start: 0 parts

Commit message: Updated board and layout, and updated gitignore
Parts:
- added C1, C2, C3: 0.1uF, SparkFun-Capacitors:0.1UF-25V(+80/-20%)(0603)
- added C4: (no value), SparkFun-Capacitors:10UF-25V-20%(PTH)KIT
- added C5: 680uF, SparkFun-Capacitors:CAP_POLPTH2
- added C6: 680 uF, SparkFun-Capacitors:CAP_POLPTH2
- added C7: 220uF, SparkFun-Capacitors:CAP_POLPTH2
- added C8: 220 uF, SparkFun-Capacitors:CAP_POLPTH2
- added D1, D2: 1N5824, SparkFun-DiscreteSemi:DIODEPTH
- added FRAME2: FRAME-LEDGER, SparkFun-Aesthetics:FRAME-LEDGER
- added JP1, JP2, JP3: (no value), SparkFun-Connectors:M022.54MM_SCREWTERM
- added L1, L2: 33 uH, SparkFun-Passives:INDUCTOR0603
- added R1, R2, R3, R4, R5: 4.7K, SparkFun-Resistors:4.7KOHM-1/10W-1%(0603)
- added R6, R8, R9: 10K, SparkFun-Resistors:10KOHM-1/10W-1%(0603)0603
- added SJ1, SJ2: JUMPER-PAD-2-NO, SparkFun-Passives:JUMPER-PAD-2-NO
- added U$1: BEAGLE_BONE_BLACK_CAPE, SparkFun-Boards:BEAGLE_BONE_BLACK_CAPE
- added U$2: TB6612FNG, SparkFun-PowerIC:TB6612FNG
- added U1: EEPROM-I2CSMD, SparkFun-DigitalIC:EEPROM-I2CSMD
- added U2, U3: LM2596, psu:LM2596
Connections:
- new net 3.3V: C1.1, R1.2, R2.2, R3.2, R4.2, R5.2, U$1P9.VDD_3V3@1, U$1P9.VDD_3V3@2, U1.VCC
- new net A01: JP2.1, U$2.A01@1, U$2.A01@2
- new net A02: JP2.2, U$2.A02@5, U$2.A02@6
- new net AIN1: U$1P9.GPIO_123, U$2.AIN1
- new net AIN2: U$1P9.GPIO_122, U$2.AIN2
- new net B01: JP3.2, U$2.B01@11, U$2.B01@12
- new net B02: JP3.1, U$2.B02@7, U$2.B02@8
- new net BIN1: U$1P9.GPIO_121, U$2.BIN1
- new net BIN2: U$1P9.GPIO_120, U$2.BIN2
- new net GND: C1.2, C2.2, C3.2, C4.-, C5.-, C6.-, C7.-, C8.-, D1.A, D2.A, JP1.1, R6.1, R9.1, SJ1.1, SJ2.1, U$1P8.DGND@1, U$1P8.DGND@2, U$1P9.DGND@1, U$1P9.DGND@2, U$1P9.DGND@3, U$1P9.DGND@4, U$1P9.DGND@5, U$1P9.DGND@6, U$2.GND, U$2.PGND1@3, U$2.PGND1@4, U$2.PGND2@10, U$2.PGND2@9, U1.VSS, U2.GND@1, U2.GND@2, U2.ON/OFF, U3.GND@1, U3.GND@2, U3.ON/OFF
- new net N$1: R3.1, U1.A0
- new net N$2: R2.1, SJ2.2, U1.A1
- new net N$3: R1.1, SJ1.2, U1.A2
- new net N$4: R8.1, R9.2, U$1P9.AIN1
- new net N$5: R6.2, U1.WP
- new net N$6: U$1P9.GPIO_48
- new net N$7: U$1P9.GPIO_31
- new net N$8: D1.C, L1.1, U2.OUT
- new net N$9: D2.C, L2.1, U3.OUT
- new net PWMA: U$1P9.GPIO_40, U$2.PWMA
- new net PWMB: U$1P9.GPIO_51, U$2.PWMB
- new net SCL: R4.1, U$1P9.I2C2_SCL, U1.SCL
- new net SDA: R5.1, U$1P9.I2C2_SDA, U1.SDA
- new net STBY: U$1P9.GPIO_117, U$2.STBY
- new net V_BATT: C5.+, C6.+, JP1.2, R8.2, U2.VIN, U3.VIN
- new net V_CPU: C2.1, C8.+, L2.2, U$1P9.SYS_5V@1, U$1P9.SYS_5V@2, U$1P9.VDD_5V@1, U$1P9.VDD_5V@2, U$2.VCC, U3.FEEDBACK
- new net V_MOTOR: C3.1, C4.+, C7.+, L1.2, U$2.VM1, U$2.VM2, U$2.VM3, U2.FEEDBACK
