File: psu-pcb/psu.sch (EAGLE design)
At the start: 31 parts, among them U1 EEPROM-I2CSMD, U2 LM2596, U3 LM2596

Commit message: Fixed board outline
Parts:
- C4: value (none) -> 10uF, 20V
Connections:
- removed net N$6: U$1P9.GPIO_48
- removed net N$7: U$1P9.GPIO_31
Changed lines of the file:
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@@
 <part name="C2" library="SparkFun-Capacitors" deviceset="0.1UF-25V(+80/-20%)(0603)" device="" value="0.1uF"/>
 <part name="C3" library="SparkFun-Capacitors" deviceset="0.1UF-25V(+80/-20%)(0603)" device="" value="0.1uF"/>
-<part name="C4" library="SparkFun-Capacitors" deviceset="10UF-25V-20%(PTH)" device="KIT"/>
+<part name="C4" library="SparkFun-Capacitors" deviceset="10UF-25V-20%(PTH)" device="KIT" value="10uF, 20V"/>
 <part name="GND19" library="SparkFun-Aesthetics" deviceset="DGND" device=""/>
 <part name="GND22" library="SparkFun-Aesthetics" deviceset="DGND" device=""/>
@@
 </segment>
 </net>
-<net name="N$6" class="0">
-<segment>
-<pinref part="U$1" gate="P9" pin="GPIO_48"/>
-<wire x1="55.88" y1="223.52" x2="43.18" y2="223.52" width="0.1524" layer="91"/>
-<label x="38.1" y="223.52" size="1.778" layer="95"/>
-</segment>
-</net>
-<net name="N$7" class="0">
-<segment>
-<pinref part="U$1" gate="P9" pin="GPIO_31"/>
-<wire x1="55.88" y1="226.06" x2="43.18" y2="226.06" width="0.1524" layer="91"/>
-<label x="38.1" y="226.06" size="1.778" layer="95"/>
-</segment>
-</net>
 <net name="N$8" class="0">
 <segment>
@@
 </sheet>
 </sheets>
+<errors>
+</errors>
 </schematic>
 </drawing>
