File: pcb/psu/psu.sch (EAGLE design)
At the start: 31 parts, among them U1 EEPROM-I2CSMD, U2 LM2596, U3 LM2596

Commit message: Updated board layout with ground pours
Parts:
- added J1: BATTERY_CONNDEANS, SparkFun-Connectors:BATTERY_CONNDEANS
Connections:
- net GND: now also J1.-
- net V_BATT: now also J1.+
Other:
- moved on the sheet: C2
Changed lines of the file:
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@@
 <part name="L2" library="SparkFun-Passives" deviceset="INDUCTOR" device="0603" value="33 uH"/>
 <part name="D2" library="SparkFun-DiscreteSemi" deviceset="DIODE" device="PTH" value="1N5824"/>
+<part name="J1" library="SparkFun-Connectors" deviceset="BATTERY_CONN" device="DEANS"/>
+<part name="SUPPLY21" library="SparkFun-Aesthetics" deviceset="V_BATT" device=""/>
+<part name="GND12" library="SparkFun-Aesthetics" deviceset="DGND" device=""/>
 </parts>
 <sheets>
@@
 <instance part="JP2" gate="G$1" x="86.36" y="104.14"/>
 <instance part="JP3" gate="G$1" x="124.46" y="104.14"/>
-<instance part="C2" gate="G$1" x="68.58" y="35.56"/>
+<instance part="C2" gate="G$1" x="15.24" y="231.14"/>
 <instance part="C3" gate="G$1" x="53.34" y="35.56"/>
 <instance part="C4" gate="G$1" x="38.1" y="38.1"/>
-<instance part="GND19" gate="G$1" x="68.58" y="22.86"/>
+<instance part="GND19" gate="G$1" x="15.24" y="218.44"/>
 <instance part="GND22" gate="G$1" x="38.1" y="22.86"/>
 <instance part="GND20" gate="G$1" x="53.34" y="22.86"/>
-<instance part="SUPPLY18" gate="G$1" x="68.58" y="48.26"/>
+<instance part="SUPPLY18" gate="G$1" x="15.24" y="243.84"/>
 <instance part="SUPPLY19" gate="G$1" x="53.34" y="48.26"/>
 <instance part="SUPPLY20" gate="G$1" x="38.1" y="48.26"/>
@@
 <attribute name="VALUE" x="380.7714" y="165.1" size="1.778" layer="96" rot="R180"/>
 </instance>
+<instance part="J1" gate="G$1" x="177.8" y="106.68" smashed="yes">
+<attribute name="VALUE" x="154.94" y="99.06" size="1.778" layer="96"/>
+<attribute name="NAME" x="175.26" y="109.982" size="1.778" layer="95"/>
+</instance>
+<instance part="SUPPLY21" gate="G$1" x="195.58" y="111.76"/>
+<instance part="GND12" gate="G$1" x="195.58" y="96.52"/>
 </instances>
 <busses>
@@
 <pinref part="C2" gate="G$1" pin="2"/>
 <pinref part="GND19" gate="G$1" pin="GND"/>
-<wire x1="68.58" y1="33.02" x2="68.58" y2="25.4" width="0.1524" layer="91"/>
+<wire x1="15.24" y1="228.6" x2="15.24" y2="220.98" width="0.1524" layer="91"/>
 </segment>
 <segment>
@@
 <wire x1="383.54" y1="162.56" x2="383.54" y2="152.4" width="0.1524" layer="91"/>
 </segment>
+<segment>
+<pinref part="GND12" gate="G$1" pin="GND"/>
+<wire x1="195.58" y1="99.06" x2="195.58" y2="104.14" width="0.1524" layer="91"/>
+<wire x1="195.58" y1="104.14" x2="185.42" y2="104.14" width="0.1524" layer="91"/>
+<pinref part="J1" gate="G$1" pin="-"/>
+</segment>
 </net>
 <net name="N$1" class="0">
@@
 <wire x1="124.46" y1="215.9" x2="124.46" y2="208.28" width="0.1524" layer="91" style="longdash"/>
 <pinref part="SUPPLY15" gate="G$1" pin="V_BATT"/>
+</segment>
+<segment>
+<pinref part="J1" gate="G$1" pin="+"/>
+<pinref part="SUPPLY21" gate="G$1" pin="V_BATT"/>
+<wire x1="185.42" y1="106.68" x2="195.58" y2="106.68" width="0.1524" layer="91"/>
+<wire x1="195.58" y1="106.68" x2="195.58" y2="111.76" width="0.1524" layer="91"/>
 </segment>
 </net>
@@
 <pinref part="C2" gate="G$1" pin="1"/>
 <pinref part="SUPPLY18" gate="G$1" pin="V_CPU"/>
-<wire x1="68.58" y1="40.64" x2="68.58" y2="48.26" width="0.1524" layer="91"/>
-</segment>
-</net>
+<wire x1="15.24" y1="236.22" x2="15.24" y2="243.84" width="0.1524" layer="91"/>
+</segment>
+</net>
